File: mcu.kicad_pcb (KiCad board)
At the start: 2 copper layers, 31 parts, among them J1 conn_male_6, Q1 BSS138, Q2 BSS138, U1 STM8S003F3P, U2 AMS1117-5.0, U3 LM358, X1 SMD_2062, X2 PH2.0_horizontal, X3 SMD2063

Commit message: mcuprototype
Parts:
- C4: value C -> 100nF
- C5: value C -> 1uF
Connections:
- J1 pad 4: PMW_OUT -> RESET
- J1 pad 5: RESET -> PMW_OUT
Routing:
- net Net-(C1-Pad2): track 56.7 -> 48.8 mm
- net RESET: track 21.5 -> 23.8 mm
Changed lines of the file:
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@@
       (effects (font (size 0.5 0.5) (thickness 0.1)))
     )
-    (fp_text value "C" (at 0 1.68 90) (layer "F.Fab")
+    (fp_text value "1uF" (at 0 1.68 90) (layer "F.Fab")
       (effects (font (size 1 1) (thickness 0.15)))
     )
@@
       (net 13 "SWIM") (pinfunction "Pin_3") (pintype "passive"))
     (pad "4" thru_hole oval (at 0 7.62 270) (size 2 2) (drill 1) (layers *.Cu *.Mask)
-      (net 11 "PMW_OUT") (pinfunction "Pin_4") (pintype "passive"))
+      (net 12 "RESET") (pinfunction "Pin_4") (pintype "passive"))
     (pad "5" thru_hole oval (at 0 10.16 270) (size 2 2) (drill 1) (layers *.Cu *.Mask)
-      (net 12 "RESET") (pinfunction "Pin_5") (pintype "passive"))
+      (net 11 "PMW_OUT") (pinfunction "Pin_5") (pintype "passive"))
     (pad "6" thru_hole oval (at 0 12.7 270) (size 2 2) (drill 1) (layers *.Cu *.Mask)
       (net 32 "LED-") (pinfunction "Pin_6") (pintype "passive"))
@@
       (effects (font (size 0.5 0.5) (thickness 0.1)))
     )
-    (fp_text value "C" (at 0 1.68) (layer "F.Fab")
+    (fp_text value "100nF" (at 0 1.68) (layer "F.Fab")
       (effects (font (size 1 1) (thickness 0.15)))
     )
@@
   (arc (start 138.991627 81.943373) (mid 139.31605 81.7266) (end 139.698734 81.65048) (width 0.3) (layer "F.Cu") (net 1))
   (arc (start 138.027893 82.907107) (mid 137.81112 83.23153) (end 137.735 83.614214) (width 0.3) (layer "F.Cu") (net 1))
+  (segment (start 120.66 98.48) (end 120.66 100.63) (width 0.4) (layer "F.Cu") (net 2))
   (segment (start 145.915 87.575) (end 145.95 87.54) (width 0.4) (layer "F.Cu") (net 2))
   (segment (start 143.4084 89.5096) (end 142.62 89.7636) (width 0.4) (layer "F.Cu") (net 2))
+  (segment (start 120.66 100.63) (end 128.81 100.63) (width 0.4) (layer "F.Cu") (net 2))
   (segment (start 143.65 87.575) (end 144 88.35) (width 0.4) (layer "F.Cu") (net 2))
   (segment (start 144 88.35) (end 144.4 89.2625) (width 0.4) (layer "F.Cu") (net 2))
-  (segment (start 120.66 94.51) (end 120.66 98.48) (width 0.4) (layer "F.Cu") (net 2))
   (segment (start 141.72625 87.575) (end 143.47375 87.575) (width 0.4) (layer "F.Cu") (net 2))
   (segment (start 143.65 87.575) (end 145.915 87.575) (width 0.4) (layer "F.Cu") (net 2))
   (segment (start 144.4 89.2625) (end 143.4084 89.5096) (width 0.4) (layer "F.Cu") (net 2))
-  (via (at 120.66 94.51) (size 1.5) (drill 0.7) (layers "F.Cu" "B.Cu") (free) (net 2))
+  (via (at 128.81 100.63) (size 1.5) (drill 0.7) (layers "F.Cu" "B.Cu") (free) (net 2))
   (via (at 145.95 87.54) (size 1.5) (drill 0.7) (layers "F.Cu" "B.Cu") (free) (net 2))
-  (segment (start 145.8 100.61) (end 120.66 100.61) (width 0.4) (layer "B.Cu") (net 2))
+  (segment (start 146.66 93.5) (end 146.66 99.75) (width 0.4) (layer "B.Cu") (net 2))
   (segment (start 145.95 87.54) (end 145.95 92.79) (width 0.4) (layer "B.Cu") (net 2))
-  (segment (start 120.66 100.61) (end 120.66 94.51) (width 0.4) (layer "B.Cu") (net 2))
+  (segment (start 145.8 100.61) (end 128.81 100.63) (width 0.4) (layer "B.Cu") (net 2))
   (segment (start 145.95 92.79) (end 146.66 93.5) (width 0.4) (layer "B.Cu") (net 2))
   (segment (start 146.66 99.75) (end 145.8 100.61) (width 0.4) (layer "B.Cu") (net 2))
-  (segment (start 146.66 93.5) (end 146.66 99.75) (width 0.4) (layer "B.Cu") (net 2))
   (segment (start 128.475 98.599) (end 128.475 98.6) (width 0.4) (layer "F.Cu") (net 5))
   (segment (start 126.375 83.6) (end 126.45953 83.51547) (width 0.4) (layer "F.Cu") (net 5))
@@
   (via (at 133.98 86.71) (size 1.5) (drill 0.7) (layers "F.Cu" "B.Cu") (free) (net 11))
   (arc (start 138.948461 97.949002) (mid 138.949573 97.949) (end 138.950685 97.949) (width 0.4) (layer "F.Cu") (net 11))
-  (segment (start 133.98 86.71) (end 136.18 82.44) (width 0.4) (layer "B.Cu") (net 11))
-  (segment (start 136.18 82.44) (end 138.98 76.59) (width 0.4) (layer "B.Cu") (net 11))
+  (segment (start 136.44 84.25) (end 136.44 76.59) (width 0.4) (layer "B.Cu") (net 11))
+  (segment (start 133.98 86.71) (end 136.44 84.25) (width 0.4) (layer "B.Cu") (net 11))
   (segment (start 133.039 95.349) (end 131.11 93.42) (width 0.4) (layer "F.Cu") (net 12))
   (segment (start 134.0185 95.349) (end 133.039 95.349) (width 0.4) (layer "F.Cu") (net 12))
   (segment (start 131.11 93.42) (end 131.11 92.97) (width 0.4) (layer "F.Cu") (net 12))
   (via (at 131.11 92.97) (size 1.5) (drill 0.7) (layers "F.Cu" "B.Cu") (free) (net 12))
-  (segment (start 132.59 85.89) (end 136.44 76.59) (width 0.4) (layer "B.Cu") (net 12))
-  (segment (start 131.11 92.97) (end 132.59 85.89) (width 0.4) (layer "B.Cu") (net 12))
+  (segment (start 138.98 85.1) (end 138.98 76.59) (width 0.4) (layer "B.Cu") (net 12))
+  (segment (start 131.11 92.97) (end 138.98 85.1) (width 0.4) (layer "B.Cu") (net 12))
   (segment (start 141.226776 94.876777) (end 141.275 94.925) (width 0.4) (layer "F.Cu") (net 13))
   (segment (start 141.275 94.925) (end 144.731716 98.381716) (width 0.4) (layer "F.Cu") (net 13))
@@
         (xy 156.4 100.75)
         (xy 156.4 96.65)
-        (xy 157.4 95.8)
-        (xy 157.4 89.35)
+        (xy 158.33 95.8)
+        (xy 158.33 89.35)
         (xy 165.36 89.35)
       )
@@
     (polygon
       (pts
-        (xy 156.95 95.7)
+        (xy 156.77 95.7)
         (xy 155.45 96.75)
         (xy 155.45 100.75)
@@
         (xy 149.706 94.95)
         (xy 149.706 89.35)
-        (xy 156.95 89.35)
+        (xy 156.77 89.35)
       )
     )
