File: mcu.kicad_sch (KiCad schematic)
At the start: 31 parts, among them J1 conn_male_6, Q1 BSS138, Q2 BSS138, U1 STM8S003F3P, U2 AMS1117-5.0, U3 LM358, X1 SMD_2062, X2 PH2.0_horizontal, X3 SMD2063

Commit message: mcuprototype
Parts:
- C4: value C -> 100nF
- C5: value C -> 1uF
- D1: symbol Light_controller-rescue:BZX84Cxx-Diode -> Diode:1N4148W
- D2: symbol Device:D_Schottky -> Diode:1N4148W
Connections:
- net PMW_OUT: now also J1.5 (Pin_5); no longer J1.4 (Pin_4)
- net RESET: now also J1.4 (Pin_4); no longer J1.5 (Pin_5)
Changed lines of the file:
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@@
     )
   )
-  (global_label "RESET" (shape input) (at 132.842 33.401 270) (fields_autoplaced)
+  (global_label "RESET" (shape input) (at 135.382 33.401 270) (fields_autoplaced)
     (effects (font (size 0.8 0.8)) (justify right))
-    (property "Intersheet References" "${INTERSHEET_REFS}" (id 0) (at 132.792 38.54 90)
+    (property "Intersheet References" "${INTERSHEET_REFS}" (id 0) (at 135.332 38.54 90)
       (effects (font (size 0.8 0.8)) (justify right) hide)
     )
@@
     )
   )
-  (global_label "PMW_OUT" (shape input) (at 135.382 33.401 270) (fields_autoplaced)
+  (global_label "PMW_OUT" (shape input) (at 132.842 33.401 270) (fields_autoplaced)
     (effects (font (size 0.8 0.8)) (justify right))
-    (property "Intersheet References" "${INTERSHEET_REFS}" (id 0) (at 135.332 40.4448 90)
+    (property "Intersheet References" "${INTERSHEET_REFS}" (id 0) (at 132.792 40.4448 90)
       (effects (font (size 0.8 0.8)) (justify right) hide)
     )
@@
   (symbol (lib_id "Device:C") (at 153.797 51.308 0) (unit 1)
     (in_bom yes) (on_board yes)
-    (property "Reference" "C4" (id 0) (at 157.607 48.768 90))
-    (property "Value" "C" (id 1) (at 157.607 51.308 90))
+    (property "Reference" "C4" (id 0) (at 149.606 51.308 90))
+    (property "Value" "100nF" (id 1) (at 157.988 51.308 90))
     (property "Footprint" "Capacitor_SMD:C_0805_2012Metric" (id 2) (at 154.7622 55.118 0)
       (effects (font (size 1.27 1.27)) hide)
@@
     (pin "2")
   )
-  (symbol (lib_id "Light_controller-rescue:BZX84Cxx-Diode") (at 40.259 48.387 180) (unit 1)
+  (symbol (lib_id "Diode:1N4148W") (at 40.259 48.387 180) (unit 1)
     (in_bom yes) (on_board yes)
     (property "Reference" "D1" (id 0) (at 41.529 44.577 0)
@@
       (effects (font (size 1.27 1.27)) hide)
     )
-    (property "Datasheet" "https://diotec.com/tl_files/diotec/files/pdf/datasheets/bzx84c2v4.pdf" (id 3) (at 40.259 48.387 0)
+    (property "Datasheet" "https://www.vishay.com/docs/85748/1n4148w.pdf" (id 3) (at 40.259 48.387 0)
       (effects (font (size 1.27 1.27)) hide)
     )
@@
   (symbol (lib_id "Device:C") (at 122.047 102.743 180) (unit 1)
     (in_bom yes) (on_board yes)
-    (property "Reference" "C5" (id 0) (at 118.237 105.283 90))
-    (property "Value" "C" (id 1) (at 118.237 102.743 90))
+    (property "Reference" "C5" (id 0) (at 118.491 102.743 90))
+    (property "Value" "1uF" (id 1) (at 126.365 102.743 90))
     (property "Footprint" "Capacitor_SMD:C_0805_2012Metric" (id 2) (at 121.0818 98.933 0)
       (effects (font (size 1.27 1.27)) hide)
@@
     (pin "2")
   )
-  (symbol (lib_id "Device:D_Schottky") (at 65.024 76.327 0) (unit 1)
+  (symbol (lib_id "Diode:1N4148W") (at 65.024 76.327 0) (unit 1)
     (in_bom yes) (on_board yes)
     (property "Reference" "D2" (id 0) (at 66.294 81.407 0))
     (property "Value" "1N4148W" (id 1) (at 70.104 78.867 0))
-    (property "Footprint" "Diode_SMD:D_SOD-123" (id 2) (at 65.024 76.327 0)
-      (effects (font (size 1.27 1.27)) hide)
-    )
-    (property "Datasheet" "~" (id 3) (at 65.024 76.327 0)
+    (property "Footprint" "Diode_SMD:D_SOD-123" (id 2) (at 65.024 80.772 0)
+      (effects (font (size 1.27 1.27)) hide)
+    )
+    (property "Datasheet" "https://www.vishay.com/docs/85748/1n4148w.pdf" (id 3) (at 65.024 76.327 0)
       (effects (font (size 1.27 1.27)) hide)
     )
@@
     )
     (path "/62a43992-3f07-46c9-a6fb-ce70d72c51bd"
-      (reference "C4") (unit 1) (value "C") (footprint "Capacitor_SMD:C_0805_2012Metric")
+      (reference "C4") (unit 1) (value "100nF") (footprint "Capacitor_SMD:C_0805_2012Metric")
     )
     (path "/df1f2632-a359-40d3-a309-00e24d8fc5cc"
-      (reference "C5") (unit 1) (value "C") (footprint "Capacitor_SMD:C_0805_2012Metric")
+      (reference "C5") (unit 1) (value "1uF") (footprint "Capacitor_SMD:C_0805_2012Metric")
     )
     (path "/cdaa5d97-e48b-49c9-ae9a-859321938986"
